Commit message: Added line following functionality and updated robot configuration

File: urdf/robot.xacro (robot description, xacro)
@@ -1,4 +1,5 @@
 <?xml version='1.0'?>
 <robot name="robot" xmlns:xacro="http://www.ros.org/wiki/xacro">
+  <!-- Properties -->
   <xacro:property name="camera_width" value="0.02"/>
   <xacro:property name="camera_length" value="0.02"/>
@@ -12,15 +13,17 @@
   <xacro:property name="wheel_width" value="0.03"/>
   <xacro:property name="wheel_mass" value="0.025"/>
+  <!-- Includes -->
   <xacro:include filename="$(find enph353_ros_lab)/urdf/macros.xacro"/>
   <xacro:include filename="$(find enph353_ros_lab)/urdf/materials.xacro"/>
-  <link name='chassis'>
+  <!-- Chassis -->
+  <link name="chassis">
     <xacro:box_inertial name="chassis" m="${chassis_mass}" x="${chassis_length}" y="${chassis_width}" z="${chassis_height}"/>
-    <collision name='chassis_collision'>
+    <collision name="chassis_collision">
       <geometry>
         <box size="${chassis_length} ${chassis_width} ${chassis_height}"/>
       </geometry>
     </collision>
-    <visual name='chassis_visual'>
-      <origin xyz="0 0 0" rpy=" 0 0 0"/>
+    <visual name="chassis_visual">
+      <origin xyz="0 0 0" rpy="0 0 0"/>
       <geometry>
         <box size="${chassis_length} ${chassis_width} ${chassis_height}"/>
@@ -31,83 +34,127 @@
     </visual>
   </link>
-  <link name='wheel_FR'>
+  <!-- Wheels -->
+  <link name="wheel_FR">
     <xacro:cylinder_inertial name="wheel_FR" m="${wheel_mass}" r="${wheel_radius}" h="${wheel_width}"/>
-    <collision name='wheel_FR_collision'>
-      <origin xyz="0 0 0" rpy="1.5708 0 0"/>
-      <geometry>
-        <cylinder radius="${wheel_radius}" length="${wheel_width}"/>
-      </geometry>
-    </collision>
-    <visual name='wheel_FR_visual'>
-      <origin xyz="0 0 0" rpy="1.5708 0 0"/>
-      <geometry>
-        <cylinder radius="${wheel_radius}" length="${wheel_width}"/>
-      </geometry>
-    </visual>
-  </link>
-  <link name='wheel_FL'>
+    <collision name="wheel_FR_collision">
+      <origin xyz="0 0 0" rpy="1.5708 0 0"/>
+      <geometry>
+        <cylinder radius="${wheel_radius}" length="${wheel_width}"/>
+      </geometry>
+    </collision>
+    <visual name="wheel_FR_visual">
+      <origin xyz="0 0 0" rpy="1.5708 0 0"/>
+      <geometry>
+        <cylinder radius="${wheel_radius}" length="${wheel_width}"/>
+      </geometry>
+    </visual>
+  </link>
+  <link name="wheel_FL">
     <xacro:cylinder_inertial name="wheel_FL" m="${wheel_mass}" r="${wheel_radius}" h="${wheel_width}"/>
-    <collision name='wheel_FL_collision'>
-      <origin xyz="0 0 0" rpy="1.5708 0 0"/>
-      <geometry>
-        <cylinder radius="${wheel_radius}" length="${wheel_width}"/>
-      </geometry>
-    </collision>
-    <visual name='wheel_FL_visual'>
-      <origin xyz="0 0 0" rpy="1.5708 0 0"/>
-      <geometry>
-        <cylinder radius="${wheel_radius}" length="${wheel_width}"/>
-      </geometry>
-    </visual>
-  </link>
-  <link name='wheel_RR'>
+    <collision name="wheel_FL_collision">
+      <origin xyz="0 0 0" rpy="1.5708 0 0"/>
+      <geometry>
+        <cylinder radius="${wheel_radius}" length="${wheel_width}"/>
+      </geometry>
+    </collision>
+    <visual name="wheel_FL_visual">
+      <origin xyz="0 0 0" rpy="1.5708 0 0"/>
+      <geometry>
+        <cylinder radius="${wheel_radius}" length="${wheel_width}"/>
+      </geometry>
+    </visual>
+  </link>
+  <link name="wheel_RR">
     <xacro:cylinder_inertial name="wheel_RR" m="${wheel_mass}" r="${wheel_radius}" h="${wheel_width}"/>
-    <collision name='wheel_RR_collision'>
-      <origin xyz="0 0 0" rpy="1.5708 0 0"/>
-      <geometry>
-        <cylinder radius="${wheel_radius}" length="${wheel_width}"/>
-      </geometry>
-    </collision>
-    <visual name='wheel_RR_visual'>
-      <origin xyz="0 0 0" rpy="1.5708 0 0"/>
-      <geometry>
-        <cylinder radius="${wheel_radius}" length="${wheel_width}"/>
-      </geometry>
-    </visual>
-  </link>
-  <link name='wheel_RL'>
+    <collision name="wheel_RR_collision">
+      <origin xyz="0 0 0" rpy="1.5708 0 0"/>
+      <geometry>
+        <cylinder radius="${wheel_radius}" length="${wheel_width}"/>
+      </geometry>
+    </collision>
+    <visual name="wheel_RR_visual">
+      <origin xyz="0 0 0" rpy="1.5708 0 0"/>
+      <geometry>
+        <cylinder radius="${wheel_radius}" length="${wheel_width}"/>
+      </geometry>
+    </visual>
+  </link>
+  <link name="wheel_RL">
     <xacro:cylinder_inertial name="wheel_RL" m="${wheel_mass}" r="${wheel_radius}" h="${wheel_width}"/>
-    <collision name='wheel_RL_collision'>
-      <origin xyz="0 0 0" rpy="1.5708 0 0"/>
-      <geometry>
-        <cylinder radius="${wheel_radius}" length="${wheel_width}"/>
-      </geometry>
-    </collision>
-    <visual name='wheel_RL_visual'>
-      <origin xyz="0 0 0" rpy="1.5708 0 0"/>
-      <geometry>
-        <cylinder radius="${wheel_radius}" length="${wheel_width}"/>
-      </geometry>
-    </visual>
-  </link>
-  <link name='camera_link'>
-    <xacro:box_inertial name="camera_link" m="${camera_mass}" x="${camera_width}" y="${camera_length}" z="${camera_height}"/>
-    <collision name='camera_link_collision'>
-      <geometry>
-        <box size="${camera_length} ${camera_width} ${camera_height}"/>
-      </geometry>
-    </collision>
-    <visual name='camera_link_visual'>
-      <origin xyz="0 0 0" rpy=" 0 0 0"/>
-      <geometry>
-        <box size="${camera_length} ${camera_width} ${camera_height}"/>
-      </geometry>
-    </visual>
-  </link>
+    <collision name="wheel_RL_collision">
+      <origin xyz="0 0 0" rpy="1.5708 0 0"/>
+      <geometry>
+        <cylinder radius="${wheel_radius}" length="${wheel_width}"/>
+      </geometry>
+    </collision>
+    <visual name="wheel_RL_visual">
+      <origin xyz="0 0 0" rpy="1.5708 0 0"/>
+      <geometry>
+        <cylinder radius="${wheel_radius}" length="${wheel_width}"/>
+      </geometry>
+    </visual>
+  </link>
+<!-- Camera -->
+<link name="camera_link">
+  <xacro:box_inertial name="camera_link" m="${camera_mass}" x="${camera_width}" y="${camera_length}" z="${camera_height}"/>
+  <collision name="camera_link_collision">
+    <geometry>
+      <box size="${camera_length} ${camera_width} ${camera_height}"/>
+    </geometry>
+  </collision>
+  <visual name="camera_link_visual">
+    <origin xyz="0 0 0" rpy="0 0 0"/>
+    <geometry>
+      <box size="${camera_length} ${camera_width} ${camera_height}"/>
+    </geometry>
+    <inertial>
+      <mass value="1e-5"/>
+      <origin xyz="0 0 0" rpy="0 0 0"/>
+      <inertia ixx="1e-6" ixy="0" ixz="0" iyy="1e-6" iyz="0" izz="1e-6"/>
+    </inertial>
+  </visual>
+</link>
+<!-- Gazebo Plugin for Camera -->
+<gazebo reference="camera_link">
+  <sensor type="camera" name="camera1">
+    <update_rate>30.0</update_rate>
+    <camera>
+      <horizontal_fov>1.3962634</horizontal_fov>
+      <image>
+        <width>800</width>
+        <height>800</height>
+        <format>R8G8B8</format>
+      </image>
+      <clip>
+        <near>0.02</near>
+        <far>300</far>
+      </clip>
+      <noise>
+        <type>gaussian</type>
+        <mean>0.0</mean>
+        <stddev>0.007</stddev>
+      </noise>
+    </camera>
+    <plugin name="camera_controller" filename="libgazebo_ros_camera.so">
+      <alwaysOn>true</alwaysOn>
+      <updateRate>30.0</updateRate> <!-- Set to 30 Hz for real-time updates -->
+      <cameraName>robot_camera</cameraName> <!-- Make sure this name is unique -->
+      <imageTopicName>/camera/image_raw</imageTopicName> <!-- Global topic name -->
+      <cameraInfoTopicName>/camera/camera_info</cameraInfoTopicName> <!-- Global topic name -->
+      <frameName>camera_link</frameName>
+      <hackBaseline>0.07</hackBaseline>
+      <distortionK1>0.0</distortionK1>
+      <distortionK2>0.0</distortionK2>
+      <distortionK3>0.0</distortionK3>
+      <distortionT1>0.0</distortionT1>
+      <distortionT2>0.0</distortionT2>
+    </plugin>
+  </sensor>
+</gazebo>
+  <!-- Joints -->
   <joint name="wheel_FR_joint" type="continuous">
     <parent link="chassis"/>
     <child link="wheel_FR"/>
-    <origin xyz="${chassis_length/2-wheel_radius} -${chassis_width/2+wheel_width/2} 0"
-            rpy="0 0 0"/>
+    <origin xyz="${chassis_length/2-wheel_radius} -${chassis_width/2+wheel_width/2} 0" rpy="0 0 0"/>
     <axis xyz="0 1 0"/>
   </joint>
@@ -115,6 +162,5 @@
     <parent link="chassis"/>
     <child link="wheel_FL"/>
-    <origin xyz="${chassis_length/2-wheel_radius} ${chassis_width/2+wheel_width/2} 0"
-            rpy="0 0 0"/>
+    <origin xyz="${chassis_length/2-wheel_radius} ${chassis_width/2+wheel_width/2} 0" rpy="0 0 0"/>
     <axis xyz="0 1 0"/>
   </joint>
@@ -122,6 +168,5 @@
     <parent link="chassis"/>
     <child link="wheel_RR"/>
-    <origin xyz="-${chassis_length/2-wheel_radius} -${chassis_width/2+wheel_width/2} 0"
-            rpy="0 0 0"/>
+    <origin xyz="-${chassis_length/2-wheel_radius} -${chassis_width/2+wheel_width/2} 0" rpy="0 0 0"/>
     <axis xyz="0 1 0"/>
   </joint>
@@ -129,6 +174,5 @@
     <parent link="chassis"/>
     <child link="wheel_RL"/>
-    <origin xyz="-${chassis_length/2-wheel_radius} ${chassis_width/2+wheel_width/2} 0"
-            rpy="0 0 0"/>
+    <origin xyz="-${chassis_length/2-wheel_radius} ${chassis_width/2+wheel_width/2} 0" rpy="0 0 0"/>
     <axis xyz="0 1 0"/>
   </joint>
@@ -138,4 +182,5 @@
     <origin xyz="${chassis_length/2} 0 ${chassis_height/2+camera_height/2}"/>
   </joint>
+  <!-- Gazebo Materials -->
   <gazebo reference="chassis">
     <material>Gazebo/Orange</material>
@@ -156,3 +201,23 @@
     <material>Gazebo/Yellow</material>
   </gazebo>
+<gazebo>
+  <plugin name="skid_steer_drive_controller" filename="libgazebo_ros_skid_steer_drive.so">
+    <updateRate>100.0</updateRate>
+    <robotNamespace>/</robotNamespace>
+    <leftFrontJoint>wheel_FL_joint</leftFrontJoint>
+    <rightFrontJoint>wheel_FR_joint</rightFrontJoint>
+    <leftRearJoint>wheel_RL_joint</leftRearJoint>
+    <rightRearJoint>wheel_RR_joint</rightRearJoint>
+    <wheelSeparation>0.4</wheelSeparation>
+    <wheelDiameter>0.215</wheelDiameter>
+    <robotBaseFrame>chassis</robotBaseFrame>
+    <torque>20</torque>
+    <topicName>/cmd_vel</topicName> <!-- Ensure it's a global topic -->
+    <odometryTopic>/odom</odometryTopic>
+    <odometryFrame>odom</odometryFrame>
+    <publishOdom>true</publishOdom>
+    <publishWheelTF>true</publishWheelTF>
+    <broadcastTF>false</broadcastTF>
+  </plugin>
+</gazebo>
 </robot>
